File: openautopihat.brd (EAGLE design)
At the start: 100 x 58.4 mm, 136 parts, among them CN1 6p-2.54, J2 DC Power Jack, Q1 s9013, Q2 s9013, U1 MCP2515, U2 MCP2551, U3 MAX2659-DFN6, U4 MP1496DJ-LF-2, U5 L70, U6 CJA1117B-3.3, U7 TXB0108PW-TSSOP20, U8 PCF85063TP, U9 BAT54C, X1 RASPI_GPIO_AB_PIN, X2 16MHz, X4 ABS07-32.768KHZ

Commit message: As prototypes manufactured
Parts:
- removed ANT1: ACD-5036-A3-CC-S, Connector-new:ANT3-SMD-5.2X3.7X0.7MM
- removed BAT_BACKUP, RTC_SDA: RTC_SDA, Discrete-new:TP-D45MIL
- removed C14: 22uF, Discrete-new:ELECTRO-SMD-B-4.8MM
- removed C15, C48: 100nF, discrete:C0603
- removed C16, C45: 10uF, discrete:C0805
- removed C22: 22uF_16V, Discrete-new:C1206
- removed C42: 22nF, discrete:C0603
- removed C46: 10uF, Discrete-new:C1206
- removed C47: DNP, discrete:C0603
- removed GPS_PPS: blue, discrete:LED-0603
- removed L1, L6: 470R,2A, discrete:L0805
- removed L2: 10uH, Discrete-new:L5040S
- removed PWR: GREEN, Discrete:LED-0603
- removed R20: 10R, discrete:R0603
- removed R21: 100K, discrete:R0603
- removed R23: 3.3K, discrete:R0603
- removed R24: 2.7K_1%, discrete:R0603
- removed R25: 510R_1%, discrete:R0603
- removed R26: 24K, discrete:R0603
- removed R7: 1k, Discrete:0603
- removed RELAY1LED, RELAY2LED: (no value), discrete:LED-0603
- removed RTC_SCL: RTC_SCL, Discrete-new:TP-D45MIL
- removed RXD: RXD, Discrete-new:TP-D45MIL
- removed TP4: INT, Discrete-new:TP-D65/35MIL
- removed TP5: CLKOUT, Discrete-new:TP-D65/35MIL
- removed TP_3V3: VCC, Discrete-new:TP-D45MIL
- removed TP_GND: GND, Discrete-new:TP-D45MIL
- removed TXD: TXD, Discrete-new:TP-D45MIL
- removed U$37, U$38, U$39, U$40, U$41, U$42, U$43: (no value), dicons:FIDUCIAL_G10
- removed U9: BAT54C, Discrete-new:SOT-23
- added ANT2: ACD-5036-A3-CC-S, Seeed-OPL-2017-01-Antenna-akita:SMD_ANT5237
- added D5, D6: 20V-1A, Seeed-Diode:SOD-123
- added INT2, INT4, INT5: RED, Discrete:LED-0603
- added J3, J4, J5: 2p-2.54, Seeed-Connector:H2-2.54
- added R42, R43: 10R, discrete:R0603
- C10: value 22uF -> 100nf; device Discrete-new:ELECTRO-SMD-B-4.8MM -> Seeed-Capacitor:C0603
- C13: value 10uF -> CAP_SMDAL_22UF_25V; device Discrete-new:C0805 -> Seeed-OPL-2017-01-Capacitor-akita:CAP_SMD_AL_D50
- C17, C18: value 7pF -> 10pF
- C19, C25, C27: device Seeed-Capacitor:C0805 -> Seeed-Capacitor:C0603
- C20: value 10uF -> 10uf; device Discrete:C0805 -> Seeed-Capacitor:C0805
- C3, C4, C43: value 100nF -> 100nf; device Discrete:C0603 -> Seeed-Capacitor:C0603
- C5: value 22uF_25V -> CAP_SMDAL_22UF_25V; device Discrete:ELECTRO-SMD-B-4.8MM -> Seeed-OPL-2017-01-Capacitor-akita:CAP_SMD_AL_D50
- C7: value 100nF -> 1uf; device discrete:C0603 -> Seeed-Capacitor:C0603
- D1: value M7 -> 28V-5A; device Discrete:D2010 -> Seeed-Diode:DO-214AA
- POWER: value blue -> RED; device discrete:LED-0603 -> Discrete:LED-0603
- R14, R15: value 1k -> 1K; device discrete:R0603 -> Seeed-Resistor:R0603
- R17, R19: device discrete:R0603 -> Seeed-Resistor:R0603
- R2: value 10k -> 10K; device Discrete:0603 -> Seeed-Resistor:R0805
- R3: value 120R -> 100R; device Discrete:0603 -> Seeed-Resistor:R0805
- R4, R5, R6: value 1k -> 1K; device Discrete:0603 -> Seeed-Resistor:R0603
- R8, R9: value 15R -> 10R
- STATUS: value blue -> BLUE; device discrete:LED-0603 -> Discrete:LED-0603
- U4: value MP1496DJ-LF-2 -> (none); device template:TSOT23-8 -> Seeed-IC:TO-220
- moved CHANNEL2 80.9 mm to (8.89, 59.7), turned to 0 degrees
- moved D1 66.3 mm to (15.2, 16.5)
- moved C25 65.3 mm to (87.6, 50.8)
- moved U6 63.1 mm to (78.0, 10.4)
- moved R28 61.9 mm to (71.1, 45.7), turned to 180 degrees
- moved CHANNEL1 61.5 mm to (8.89, 43.2), turned to 0 degrees
- moved RELAY2 60.5 mm to (24.1, 57.1), turned to 180 degrees
- moved R27 59.9 mm to (71.1, 47.0), turned to 180 degrees
- moved STATUS 59.5 mm to (47.1, 2.16)
- moved J2 57.4 mm to (27.9, 0.00), turned to 0 degrees
- moved Q2 56.6 mm to (40.6, 58.4)
- moved C11 56.5 mm to (81.3, 55.2)
- moved POWER 56.5 mm to (54.7, 2.29)
- moved Q1 51.2 mm to (40.6, 43.2)
- moved C1 49.6 mm to (21.6, 24.1), turned to 90 degrees
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Connections:
- removed net 5V1: C14.+, U6.3
- removed net N$1: PWR.+, R7.1
- removed net N$14: C48.2, U4.7
- removed net N$18: C7.1, L2.1, U4.3
- removed net N$21: C42.2, U4.1
- removed net N$22: R20.1, U4.5
- removed net N$24: C7.2, R20.2
- removed net N$25: R23.1, U4.8
- removed net N$27: C47.2, R23.2, R24.2, R25.2
- removed net N$28: R21.1, R26.1, U4.6
- removed net OUT1: C13.2, C45.2, C46.2, C47.1, L2.2, L6.1, R24.1
- removed net PWR_IN: C10.+, C22.1, L1.2, R21.2, U4.2
- new net N$30: P1.1, R3.2
- new net N$45: R42.2, R43.1
- net !RTC_INT: no longer TP4.P1
- net +3V: now also D6.+, R40.2; no longer TP_3V3.T, U9.1
- net +5V: now also C10.2, C13.P$P, U4.3, U6.3; no longer C15.1, C16.1, L6.2, R7.2
- net BAT_BACKUP: now also D5.+; no longer BAT_BACKUP.T, U9.2
- net CANH: no longer P1.1, R3.1
- net CANL: now also R43.2; no longer R3.2
- net GND: now also ANT2.GND1, ANT2.GND2, C10.1, C13.P$M, C5.P$M, C7.1, INT2.-, J3.1, J4.1, J5.1, R41.1, U4.2, U4.HEAT; no longer ANT1.2, ANT1.3, C10.-, C13.1, C14.-, C15.2, C16.2, C22.2, C42.1, C45.1, C46.1, C48.1, C5.-, GPS_PPS.-, PWR.-, R25.1, R26.2, TP_GND.T, U4.4
- net N$10: now also J4.2
- net N$11: now also R3.1, R42.1; no longer POWER.+, R19.2
- net N$12: now also INT5.-; no longer RELAY1LED.-
- net N$13: now also INT4.-; no longer RELAY2LED.-
- net N$26: now also C7.2, U4.1; no longer L1.1
- net N$29: now also J3.2, POWER.+, R19.2; no longer R40.2
- net N$32: now also ANT2.FEED; no longer ANT1.1
- net N$49: now also D5.-, D6.-; no longer U9.3
- net N$9: now also INT2.+, J5.2; no longer GPS_PPS.+
- net RELAY1: now also INT5.+; no longer RELAY1LED.+
- net RELAY2: now also INT4.+; no longer RELAY2LED.+
- net RTC_CLKOUT: no longer TP5.P1
- net RTC_SCL: no longer RTC_SCL.T
- net RTC_SDA: no longer RTC_SDA.T
- net RXD1: no longer RXD.T
- net TXD1: no longer TXD.T
- net V+: now also C5.P$P; no longer C5.+
Routing:
- net +5V: track 0.00 -> 248.0 mm, vias 0 -> 6
- net +3V: track 0.00 -> 158.5 mm, vias 0 -> 10
- net RST_N: track 0.00 -> 109.5 mm, vias 0 -> 2
- net RFIDRX: track 0.00 -> 105.6 mm, vias 0 -> 2
- net RFIDTX: track 0.00 -> 70.3 mm, vias 0 -> 1
- net RELAY2: track 0.00 -> 57.0 mm
- net RELAY1: track 0.00 -> 57.0 mm
- net CAN_MOSI: track 0.00 -> 54.6 mm
- net RTC_SDA: track 0.00 -> 53.1 mm, vias 0 -> 3
- net CAN_SCK: track 0.00 -> 52.4 mm, vias 0 -> 2
- net POWERLED: track 0.00 -> 50.8 mm, vias 0 -> 1
- net GPS_UART0_RX: track 0.00 -> 45.7 mm
- net CANL: track 0.00 -> 44.7 mm, vias 0 -> 1
- net RTC_SCL: track 0.00 -> 42.3 mm, vias 0 -> 3
- net CAN_CS: track 0.00 -> 40.9 mm, vias 0 -> 2
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- added copper zone on layer 1, net GND
- added copper zone on layer 16, net GND
Other:
- board size 100 x 58.4 mm -> 100 x 67.3 mm
- board text added: "15V Max"
- board text added: "CAN to Vehicle"
- board text added: "External Control"
- board text added: "J.Devine CERN OHL v1.2"
- board text added: "OpenAuto.ch Car Sharing"
- board text added: "RFID UART"
- board text added: "Raspberry Pi Header"
- board text added: "github.com/pingud98/OpenAutoChPiHat"
