File: openautopihat.sch (EAGLE design)
At the start: 127 parts, among them CN1 6p-2.54, J2 DC Power Jack, Q1 s9013, Q2 s9013, Q3 2N7002, Q4 2N7002, U1 MCP2515, U2 MCP2551, U3 ATMEGA328P, U4 MP1496DJ-LF-2, U6 CJA1117B-3.3, U7 TXB0108PW-TSSOP20, U8 PCF85063TP, U9 BAT54C, X1 RASPI_BOARD_B+#_HDC, X2 16MHz, X3 16MHz, X4 ABS07-32.768KHZ

Commit message: Schematic revised & completed. Layout in progress
Parts:
- removed C41: 100nF, discrete:C-0603
- removed CS, MISO, MOSI, SCK: (no value), Discrete:PAD-JUMPER-3P-40*40
- removed I2C, SERIAL: (no value), Connector:TWIG-4P-2.0-2.0
- removed L: blue, discrete:LED'0603'
- removed PWR1: GREEN, discrete:LED'0603'
- removed Q3, Q4: 2N7002, Seeed-Transistor:SMD-MOSFET-N-CH-60V-300MA-LOGIC-LEVEL-FET-2N7002(SOT-23)
- removed RESET: BUTTON-4P-REINFORCE, discrete:BUTTON-4P-REINFORCE'TS-1188E'
- removed RST: RED, discrete:LED'0603'
- removed TP1, TP2, TP3: (no value), Discrete:PAD-TEST-POINT'4545'
- removed TP10: RTC_SCL, Discrete-new:TEST-POINT'4545'
- removed TP12: VCC, Discrete-new:TEST-POINT'4545'
- removed TP13: GND, Discrete-new:TEST-POINT'4545'
- removed V_OBD: (no value), Discrete:SWITCH-2CH-6P
- removed X3: 16MHz, discrete:CRYSTAL'5032'
- added ANT1: ACD-5036-A3-CC-S, Connector-new:ANTENNA-ACD5036
- added C23: 33nf, Seeed-Capacitor:CERAMIC-33NF-50V-10%-X7R(0603)
- added C24, C26, C28: 10uf, Seeed-Capacitor:CERAMIC-10UF-25V-10%-X5R(0805)
- added C25, C27, C29: 100nf, Seeed-Capacitor:CERAMIC-100NF-50V-10%-X7R(0805)
- added GPS_PPS, POWER, STATUS: blue, discrete:LED'0603'
- added L5: 4.7NH-300MA, Seeed-Inductor:SMD-INDUCTOR-4.7NH-0.3NH-300MA(0402)
- added L7: DNP, Discrete-new:INDUCTOR/FERRITE-BEAD-0201
- added R34, R35, R36, R37: 0R, Seeed-Resistor:SMD-RES-0R-5%-1/10W(0603)
- added R38, R39, R40, R41: DNP, discrete:R-0603
- added RXD: RXD, Discrete-new:TEST-POINT'4545'
- added TXD: TXD, Discrete-new:TEST-POINT'4545'
- C11, C9: value 100nF -> DNP; device discrete:C-0603 -> Discrete-new:CAP-0201
- C12: value 10uF -> 100pf; device discrete:C-0805 -> Seeed-Capacitor:CERAMIC-100PF-50V-5%-NPO(0603)
- C19: value 100nF -> 100nf; device Discrete-new:CAP-0402 -> Seeed-Capacitor:CERAMIC-100NF-50V-10%-X7R(0805)
- C6, C8: value 22pF -> 100pf; device discrete:C-0603 -> Seeed-Capacitor:CERAMIC-100PF-50V-5%-NPO(0603)
- R18: value 10K -> 100R; device discrete:R-0603 -> Seeed-Resistor:SMD-RES-100R-5%-1/8W(0805)
- R22: value 0R -> 100R; device discrete:R-0603 -> Seeed-Resistor:SMD-RES-100R-5%-1/8W(0805)
- R27, R28: value 10k -> DNP; device Discrete:R-0603 -> Discrete-new:RES-0201
- R29, R30: value 10k -> 0R; device Discrete:R-0603 -> Seeed-Resistor:SMD-RES-0R-5%-1/10W(0603)
- R31, R32, R33: device Discrete-new:RES-0402 -> Seeed-Resistor:SMD-RES-10K-1%-1/8W(0805)
- U3: value ATMEGA328P -> MAX2659-DFN6; device ICs_v54:MEGA8 -> IC-new:AMPLIFIER-MAX2659
- U5: value (none) -> L70; device Seeed-OPL-2017-01-Sensor-camilo:L70-M39 -> moudle-new:MOUDLE-GPS-L70-HARDWARE
- X1: value RASPI_BOARD_B+#_HDC -> RASPI_GPIO_AB_PIN; device raspberrypi_bastelstube_v13:RASPI_BOARD_B+#_HDC -> raspberrypi_bastelstube_v13:RASPI_GPIO_AB_PIN
- renumbered LED1 to RELAY1LED, LED2 to RELAY2LED, TP11 to BAT_BACKUP, TP6 to RTC_SCL, TP7 to RTC_SDA, TP8 to TP_3V3, TP9 to TP_GND
Connections:
- removed net +3V3: Q3.G, Q4.G, R28.2, R30.2
- removed net 3V3: C20.1, C43.2, U6.OUT
- removed net 5V: C3.1, C4.1, D2.-, D3.-, I2C.3, R2.2, R4.2, R5.2, R6.2, R7.2, RELAY1.V+, RELAY2.V+, SERIAL.3, U1.VDD, U2.VDD
- removed net ADC4: I2C.2
- removed net ADC5: I2C.1
- removed net AREF: U3.AREF
- removed net CLKOUT: TP5.T, U8.CLKOUT
- removed net CS: CS.C, U1.!CS
- removed net CS_A: CS.R
- removed net CS_B: CS.L
- removed net EXT_PWR: D4.+, J2.+, VIN.T
- removed net INT: INT.-, U1.!INT
- removed net IO0: SERIAL.1
- removed net IO1: SERIAL.2
- removed net IOREF: R22.2
- removed net MISO: MISO.C, U1.SO
- removed net MISO_A: MISO.L
- removed net MISO_B: MISO.R
- removed net MOSI: MOSI.C, U1.SI
- removed net MOSI_A: MOSI.L
- removed net MOSI_B: MOSI.R
- removed net PB0: U3.PB0(ICP)
- removed net PB1: U3.PB1(OC1A)
- removed net PB2: U3.PB2(SS/OC1B)
- removed net PB3/MOSI: U3.PB3(MOSI/OC2)
- removed net PB4/MISO: U3.PB4(MISO)
- removed net PB5/SCK: R19.1, U3.PB5(SCK)
- removed net PC0: U3.PC0(ADC0)
- removed net PC1: U3.PC1(ADC1)
- removed net PC2: U3.PC2(ADC2)
- removed net PC3: U3.PC3(ADC3)
- removed net PC4/SDA: U3.PC4(ADC4/SDA)
- removed net PC5/SCL: U3.PC5(ADC5/SCL)
- removed net PD0/RX: U3.PD0(RXD)
- removed net PD1/TX: U3.PD1(TXD)
- removed net PD2/INT0: U3.PD2(INT0)
- removed net PD3/INT1: U3.PD3(INT1)
- removed net PD4: U3.PD4(XCK/T0)
- removed net PD5: U3.PD5(T1)
- removed net PD6: U3.PD6(AIN0)
- removed net PD7: U3.PD7(AIN1)
- removed net RESET: R18.2, RESET.1, RST.-, U3.PC6(/RESET)
- removed net RPI-SCL: Q3.S, R28.1
- removed net RPI-SDA: Q4.S, R30.1
- removed net SCK: SCK.C, U1.SCK
- removed net SCK_A: SCK.L
- removed net SCK_B: SCK.R
- removed net SCL-BOARD: Q3.D, R27.1
- removed net SDA-BOARD: Q4.D, R29.1
- removed net VCC: C11.2, C12.1, C15.1, C16.1, C21.2, C41.2, C9.2, L6.2, R16.1, R17.1, R18.1, R22.1, R27.2, R29.2, R31.2, R32.1, R33.2, TP_3V3.T, U3.AVCC, U3.VCC@1, U3.VCC@2, U9.P$1
- removed net VIN: V_OBD.COM1, V_OBD.COM2
- removed net XTAL1: C6.2, U3.PB6(XTAL1/TOSC1), X3.2
- removed net XTAL2: C8.2, U3.PB7(XTAL2/TOSC2), X3.1
- new net +3V: C20.1, C21.2, C24.1, C25.1, C26.1, C27.1, C43.2, CN1.1, R29.1, R31.2, R32.1, R33.2, R38.2, TP_3V3.T, U5.VCC, U6.OUT, U7.VCCB, U9.P$1
- new net +5V: C15.1, C16.1, C28.1, C29.1, C3.1, C4.1, D2.-, D3.-, L6.2, R2.2, R4.2, R5.2, R6.2, R7.2, RELAY1.V+, RELAY2.V+, U1.VDD, U2.VDD, U7.OE, U7.VCCA, X1.5V0, X1.N.C.0
- new net 3CAN_CS: U7.B1, X1.SPI_CE0
- new net 3CAN_INT: U7.B5, X1.GPIO18
- new net 3CAN_MISO: U7.B3, X1.SPI_MOSI
- new net 3CAN_MOSI: U7.B2, X1.SPI_MISO
- new net 3CAN_SCK: U7.B4, X1.SPI_SCLK
- new net 3RELAY1: U7.B6, X1.GPIO23
- new net 3RELAY2: U7.B7, X1.GPIO24
- new net ANTON: R18.2, U5.ANTON
- new net CAN_CS: U1.!CS, U7.A1
- new net CAN_INT: INT.-, U1.!INT, U7.A5
- new net CAN_MISO: U1.SO, U7.A3
- new net CAN_MOSI: U1.SI, U7.A2
- new net CAN_SCK: U1.SCK, U7.A4
- new net GPS_1PPS: R16.1, R34.1
- new net GPS_STANDBY: R30.1, X1.GPIO25
- new net GPS_UART0_RX: R35.1, X1.TXD
- new net GPS_UART0_TX: R36.1, X1.RXD
- new net N$31: C6.1, C8.2, C9.2
- new net N$32: ANT1.D, C11.2, C6.2
- new net N$33: L5.1, L7.2, U3.RFIN
- new net N$34: C8.1, L5.2
- new net N$35: R18.1, U3.!SHDN
- new net N$36: C12.1, C23.1, R22.1, U3.VCC
- new net N$37: R27.1, U5.RESERVED
- new net N$38: R28.1, U5.RESERVED1
- new net N$39: R29.2, U5.V_BCKP
- new net N$42: R30.2, U5.STANDBY
- new net N$43: R34.2, U5.1PPS
- new net N$44: R37.2, U5.RESET
- new net POWERLED: R19.1, X1.N.C.3
- new net RFIDRX: CN1.4, R17.1, X1.GPIO27
- new net RFIDTX: CN1.3, X1.GPIO17
- new net RF_IN: U3.RFOUT, U5.RF_IN
- new net RTC_CLKOUT: TP5.T, U8.CLKOUT, X1.GPIO22
- new net RXD1: R35.2, RXD.T, U5.RXD1
- new net TXD1: R36.2, TXD.T, U5.TXD1
- new net VCC_RF: R22.2, U5.VCC_RF
- net !RTC_INT: now also X1.SPI_CE1
- net GND: now also ANT1.GND1, ANT1.GND2, C23.2, C24.2, C25.2, C26.2, C27.2, C28.2, C29.2, CN1.2, GPS_PPS.-, L7.1, POWER.-, R27.2, R28.2, R39.1, STATUS.-, U3.GND, U5.GND, U5.GND@1, U5.GND@2, U7.GND, X1.GND, X1.N.C.1, X1.N.C.2, X1.N.C.4, X1.N.C.5; no longer C41.1, C6.1, C8.1, I2C.4, L.-, PWR1.-, RESET.2, RESET.S1, RESET.S2, SERIAL.4, U3.AGND, U3.GND@2, U3.HEAT
- net N$10: now also STATUS.+; no longer PWR1.+
- net N$11: now also POWER.+; no longer L.+
- net N$29: now also R40.2; no longer U7.OE
- net N$9: now also GPS_PPS.+; no longer RST.+
- net RELAY1: now also U7.A6
- net RELAY2: now also U7.A7
- net RST_N: now also R37.1, X1.GPIO04
- net RTC_SCL: now also R38.1, R39.2, X1.SCL
- net RTC_SDA: now also R40.1, R41.2, X1.SDA
- net V+: now also D4.+, J2.+, VIN.T; no longer V_OBD.CH1A, V_OBD.CH2A
Other:
- note added: "3.3V to 5V Level Converter"
- note added: "Designed by James Devine"
- note added: "GPS MODULE based on SEEED XADOW GPS"
- note added: "Impedance of RF trace should be controlled by 50 ohm and the length should be kept as short as possible."
- note added: "LEDs"
- note added: "Licensed under the CERN OHL V1.2"
- note added: "Minimum Pi Header (26 pins)"
- note added: "Note RFID is TX only, therefore we use this pin for a status LED"
- note added: "Openauto Pi Hat V1"
- note added: "Optional pull ups/downs for I2C bus"
- note added: "Power supply block (5V and 3.3V) borrowed from an Arduino Pi Hat"
- note added: "Prototype assembly in progress 16 aug 17"
- note added: "http://github.com/pingud98/OpenAutoChPiHat"
- note removed: "5V tolerant, connect to D11."
- moved on the sheet: C11, C9, CN1, R16, R17, R19, R27, R28, TP5, U5, U7

Commit message: As prototypes manufactured
Parts:
- removed ANT1: ACD-5036-A3-CC-S, Connector-new:ANTENNA-ACD5036
- removed BAT_BACKUP, RTC_SDA: RTC_SDA, Discrete-new:TEST-POINT'4545'
- removed C14: 22uF, Discrete-new:CAP-POLAR-ELECTRO-B
- removed C15, C48: 100nF, discrete:C-0603
- removed C16, C45: 10uF, discrete:C-0805
- removed C22: 22uF_16V, Discrete-new:CAP-1206
- removed C42: 22nF, discrete:C-0603
- removed C46: 10uF, Discrete-new:CAP-1206
- removed C47: DNP, discrete:C-0603
- removed GPS_PPS: blue, discrete:LED'0603'
- removed L1, L6: 470R,2A, discrete:L'0805'
- removed L2: 10uH, Discrete-new:INDUCTOR/FERRITE-BEAD5040S
- removed PWR: GREEN, Discrete:LED'0603'
- removed R20: 10R, discrete:R-0603
- removed R21: 100K, discrete:R-0603
- removed R23: 3.3K, discrete:R-0603
- removed R24: 2.7K_1%, discrete:R-0603
- removed R25: 510R_1%, discrete:R-0603
- removed R26: 24K, discrete:R-0603
- removed R7: 1k, Discrete:R-0603
- removed RELAY1LED, RELAY2LED: (no value), discrete:LED'0603'
- removed RTC_SCL: RTC_SCL, Discrete-new:TEST-POINT'4545'
- removed RXD: RXD, Discrete-new:TEST-POINT'4545'
- removed TP4: INT, Discrete-new:TEST-POINT
- removed TP5: CLKOUT, Discrete-new:TEST-POINT
- removed TP_3V3: VCC, Discrete-new:TEST-POINT'4545'
- removed TP_GND: GND, Discrete-new:TEST-POINT'4545'
- removed TXD: TXD, Discrete-new:TEST-POINT'4545'
- removed U9: BAT54C, Discrete-new:DIODE-BAT54C
- added ANT2: ACD-5036-A3-CC-S, Seeed-OPL-2017-01-Antenna-akita:ACD-5036-A3-CC-S
- added D5, D6: 20V-1A, Seeed-Diode:SMD-DIODE-SCHOTTKY-20V-1A(SOD-123)
- added INT2, INT4, INT5: RED, Discrete:LED'0603'
- added J3, J4, J5: 2p-2.54, Seeed-Connector:DIP-BLACK-MALE-HEADER-VERT(2P-2.54)
- added R42, R43: 10R, discrete:R-0603
- C10: value 22uF -> 100nf; device Discrete-new:CAP-POLAR-ELECTRO-B -> Seeed-Capacitor:CERAMIC-100NF-50V-10%-X7R(0603)
- C13: value 10uF -> CAP_SMDAL_22UF_25V; device Discrete-new:CAP-0805 -> Seeed-OPL-2017-01-Capacitor-akita:CAP_SMDAL_22UF_25V
- C17, C18: value 7pF -> 10pF
- C19, C25, C27: device Seeed-Capacitor:CERAMIC-100NF-50V-10%-X7R(0805) -> Seeed-Capacitor:CERAMIC-100NF-50V-10%-X7R(0603)
- C20: value 10uF -> 10uf; device Discrete:C-0805 -> Seeed-Capacitor:CERAMIC-10UF-25V-10%-X5R(0805)
- C3, C4, C43: value 100nF -> 100nf; device Discrete:C-0603 -> Seeed-Capacitor:CERAMIC-100NF-50V-10%-X7R(0603)
- C5: value 22uF_25V -> CAP_SMDAL_22UF_25V; device Discrete:CAP-ELECTRO-B -> Seeed-OPL-2017-01-Capacitor-akita:CAP_SMDAL_22UF_25V
- C7: value 100nF -> 1uf; device discrete:C-0603 -> Seeed-Capacitor:CERAMIC-1UF-25V-10%-X7R(0603)
- D1: value M7 -> 28V-5A; device Discrete:D-SMA -> Seeed-Diode:SMD-DIODE-SCHOTTKY-28V-5A(DO-214AA)
- POWER: value blue -> RED; device discrete:LED'0603' -> Discrete:LED'0603'
- R14, R15: value 1k -> 1K; device discrete:R-0603 -> Seeed-Resistor:SMD-RES-1K-1%-1/10W(0603)
- R17, R19: device discrete:R-0603 -> Seeed-Resistor:SMD-RES-1K-1%-1/10W(0603)
- R2: value 10k -> 10K; device Discrete:R-0603 -> Seeed-Resistor:SMD-RES-10K-1%-1/8W(0805)
- R3: value 120R -> 100R; device Discrete:R-0603 -> Seeed-Resistor:SMD-RES-100R-5%-1/8W(0805)
- R4, R5, R6: value 1k -> 1K; device Discrete:R-0603 -> Seeed-Resistor:SMD-RES-1K-1%-1/10W(0603)
- R8, R9: value 15R -> 10R
- STATUS: value blue -> BLUE; device discrete:LED'0603' -> Discrete:LED'0603'
- U4: value MP1496DJ-LF-2 -> (none); device template:MP1496DJ -> Seeed-IC:PMIC-ST-L7805CV(TO-220)
Connections:
- removed net 5V1: C14.+, U6.IN
- removed net N$1: PWR.+, R7.1
- removed net N$14: C48.2, U4.VCC
- removed net N$18: C7.1, L2.1, U4.SW
- removed net N$21: C42.2, U4.SS
- removed net N$22: R20.1, U4.BS
- removed net N$24: C7.2, R20.2
- removed net N$25: R23.1, U4.FB
- removed net N$27: C47.2, R23.2, R24.2, R25.2
- removed net N$28: R21.1, R26.1, U4.EN/SYNC
- removed net OUT1: C13.2, C45.2, C46.2, C47.1, L2.2, L6.1, R24.1
- removed net PWR_IN: C10.+, C22.1, L1.2, R21.2, U4.IN
- new net N$30: P1.1, R3.2
- new net N$45: R42.2, R43.1
- net !RTC_INT: no longer TP4.T
- net +3V: now also D6.+, R40.2; no longer TP_3V3.T, U9.P$1
- net +5V: now also C10.2, C13.P$P, U4.OUT, U6.IN; no longer C15.1, C16.1, L6.2, R7.2
- net BAT_BACKUP: now also D5.+; no longer BAT_BACKUP.T, U9.P$2
- net CANH: no longer P1.1, R3.1
- net CANL: now also R43.2; no longer R3.2
- net GND: now also ANT2.GND1, ANT2.GND2, C10.1, C13.P$M, C5.P$M, C7.1, INT2.-, J3.1, J4.1, J5.1, R41.1; no longer ANT1.GND1, ANT1.GND2, C10.-, C13.1, C14.-, C15.2, C16.2, C22.2, C42.1, C45.1, C46.1, C48.1, C5.-, GPS_PPS.-, PWR.-, R25.1, R26.2, TP_GND.T
- net N$10: now also J4.2
- net N$11: now also R3.1, R42.1; no longer POWER.+, R19.2
- net N$12: now also INT5.-; no longer RELAY1LED.-
- net N$13: now also INT4.-; no longer RELAY2LED.-
- net N$26: now also C7.2, U4.IN; no longer L1.1
- net N$29: now also J3.2, POWER.+, R19.2; no longer R40.2
- net N$32: now also ANT2.FEED; no longer ANT1.D
- net N$49: now also D5.-, D6.-; no longer U9.P$3
- net N$9: now also INT2.+, J5.2; no longer GPS_PPS.+
- net RELAY1: now also INT5.+; no longer RELAY1LED.+
- net RELAY2: now also INT4.+; no longer RELAY2LED.+
- net RTC_CLKOUT: no longer TP5.T
- net RTC_SCL: no longer RTC_SCL.T
- net RTC_SDA: no longer RTC_SDA.T
- net RXD1: no longer RXD.T
- net TXD1: no longer TXD.T
- net V+: now also C5.P$P; no longer C5.+
Other:
- note removed: "Power supply block (5V and 3.3V) borrowed from an Arduino Pi Hat"
- moved on the sheet: BAT1, C1, C11, C12, C17, C18, C19, C2, C21, C23, C24, C25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
