File: openautopihatv1point1.sch (EAGLE design)
At the start: 98 parts, among them CN1 6p-2.54, CN2 6p-2.54, J2 DC Power Jack, J3 2p-2.54, J4 2p-2.54, J5 2p-2.54, J6 2p-2.54, J7 2p-2.54, Q1 s9013, Q2 s9013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

Commit message: Version 1.1 design completed
Parts:
- removed D4: 1N5819, discrete:D'DO-214AC'
- removed J4, J5, J6, J7: 2p-2.54, Seeed-Connector:DIP-BLACK-MALE-HEADER-VERT(2P-2.54)
- removed VIN: (no value), discrete:PAD-TEST-POINT'4545'
- added C16, C22: 100nf, Seeed-Capacitor:CERAMIC-100NF-50V-10%-X7R(0603)
- added C23, C24: DNP, Seeed-Capacitor:CERAMIC-1NF-50V-5%-C0G(0603)
- added CN3: 6p-2.54, Seeed-Connector:DIP-BLACK-FEMALE-HEADER-VERT(6P-2.54)
- added R24: 0R, Seeed-Resistor:SMD-RES-0R-5%-1/10W(0603)
- added STATUS1: BLUE, Discrete:LED'0603'
- added U3: MMA7660FCR1, Seeed-Sensor:MOTION/POSITION-MMA7660FCR1(DFN10)
- C17, C18: value 10pF -> 10pf; device Discrete-new:CAP-0402 -> Seeed-Capacitor:CERAMIC-10PF-50V-5%-NPO(0603)
- C21: value 10uF -> 10uf; device Discrete-new:CAP-0805 -> Seeed-Capacitor:CERAMIC-10UF-25V-10%-X5R(0805)
- J1: device Connector:DB9'MEAL' -> SparkFun-Connectors:DB9MALE
- J2: value DC Power Jack -> (none); device For_Test_Albert:DC-044 -> Connector:SCREW-TERMINAL-2P5.0
- J3: value 2p-2.54 -> 4p-2.54; device Seeed-Connector:DIP-BLACK-MALE-HEADER-VERT(2P-2.54) -> Seeed-Connector:DIP-BLACK-FEMALE-HEADER-VERT(4P-2.54)
- R16: value 1K -> 1K 1/10W; device discrete:R-0603 -> Seeed-Resistor:SMD-RES-1K-5%-1/10W(0603)
- R17: value 1K -> 100R; device Seeed-Resistor:SMD-RES-1K-1%-1/10W(0603) -> Seeed-Resistor:SMD-RES-100R-5%-1/10W(0603)
- R18, R2, R20, R23, R31, R32, R33: value 10K -> 10K 1/10W; device Seeed-Resistor:SMD-RES-10K-1%-1/8W(0805) -> Seeed-Resistor:SMD-RES-10K-5%-1/10W(0603)
- R3: device Seeed-Resistor:SMD-RES-100R-5%-1/8W(0805) -> Seeed-Resistor:SMD-RES-100R-5%-1/10W(0603)
- R38, R40: value DNP -> 3.9k
- U4: value (none) -> CJ78M05-to252; device Seeed-IC:PMIC-ST-L7805CV(TO-220) -> Seeed-IC:PMIC-CJ78M05(TO-252)
- renumbered INT2 to PPS, INT4 to R2LED, INT5 to R1LED
Connections:
- removed net CAN_INT: INT.-, X1.GPIO18
- removed net N$21: CN2.4
- removed net N$26: C7.2, D4.-, U4.IN
- removed net N$27: R20.1
- removed net RTC_CLKOUT: U8.CLKOUT, X1.GPIO22
- new net ACCELINT: U3.!INT, X1.GPIO22
- net +3V: now also C16.2, C22.2, J3.P$1, U3.AVDD, U3.DVDD
- net +5V: now also CN2.5
- net CAN_!INT: now also INT.-, X1.GPIO18
- net GND: now also C16.1, C22.1, C23.1, C24.1, CN2.4, J2.2, J3.P$2, R20.1, STATUS1.-, U3.AVSS, U3.DVSS, U3.RESERVED; no longer J1.10, J1.11, J2.-, J2.CDN, J3.1, J4.1, J5.1, J6.1, J7.1
- net N$1: no longer J6.2
- net N$10: now also STATUS1.+; no longer J4.2
- net N$14: now also C24.2, R24.1; no longer X3.1
- net N$18: now also C23.2, R24.2, X3.1; no longer CN2.5
- net N$25: no longer J7.2
- net N$29: no longer J3.2
- net N$9: no longer J5.2
- net RTC_SCL: now also J3.P$3, U3.SCL
- net RTC_SDA: now also J3.P$4, U3.SDA
- net V+: now also C7.2, J2.1, U4.IN; no longer D4.+, J2.+, VIN.T
Other:
- note added: "Accelerometer"
- note added: "I2C header"
- note added: "Notes to self: Remove 0806 components Relocate OrangePi Header to middle/rotate Add accelerometer Relocate LEDS Add LED for RFID Status Add a buzzer?"
- note added: "Power supply: Vin, 5V and 3.3V rails"
- note added: "RTC Module and I2C Header"
- note added: "null connector for RDM6300"
- note removed: "Note RFID is TX only, therefore we use this pin for a status LED"
- note removed: "RTC Module"
- moved on the sheet: C10, C13, C20, C43, C6, C7, C8, C9, MODULE1, R38, R39, R40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
